File: pcb/MP3_Decoder.sch (KiCad schematic (older format))
At the start: 31 parts, among them J3 Screw_Terminal_1x04, U6 STA013, U7 CS4344, U8 PAM8403, Y2 12MHz

Commit message: Switched to nodemcu-style flashing circuitry.
Other:
- moved on the sheet: C10, C11, C12, C13, C14, C15, C16, C17, C18, C19, C20, C21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
